Commit message: set float

File: models/TR5.urdf (robot description, URDF)
Before this commit: robot TR5, 31 links, 30 joints
Links:
- link Link_ankle_l_pitch: geometry collision mesh filename=package://TR5/meshes/Link_ankle_l_pitch.STL; visual mesh filename=package://TR5/meshes/Link_ankle_l_pitch.STL
- link Link_ankle_l_roll: geometry collision mesh filename=package://TR5/meshes/Link_ankle_l_roll.STL; visual mesh filename=package://TR5/meshes/Link_ankle_l_roll.STL
- link Link_ankle_r_pitch: geometry collision mesh filename=package://TR5/meshes/Link_ankle_r_pitch.STL; visual mesh filename=package://TR5/meshes/Link_ankle_r_pitch.STL
- link Link_ankle_r_roll: geometry collision mesh filename=package://TR5/meshes/Link_ankle_r_roll.STL; visual mesh filename=package://TR5/meshes/Link_ankle_r_roll.STL
- link Link_arm_l_01: geometry collision mesh filename=package://TR5/meshes/Link_arm_l_01.STL; visual mesh filename=package://TR5/meshes/Link_arm_l_01.STL
- link Link_arm_l_02: geometry collision mesh filename=package://TR5/meshes/Link_arm_l_02.STL; visual mesh filename=package://TR5/meshes/Link_arm_l_02.STL
- link Link_arm_l_03: geometry collision mesh filename=package://TR5/meshes/Link_arm_l_03.STL; visual mesh filename=package://TR5/meshes/Link_arm_l_03.STL
- link Link_arm_l_04: geometry collision mesh filename=package://TR5/meshes/Link_arm_l_04.STL; visual mesh filename=package://TR5/meshes/Link_arm_l_04.STL
- link Link_arm_l_05: geometry collision mesh filename=package://TR5/meshes/Link_arm_l_05.STL; visual mesh filename=package://TR5/meshes/Link_arm_l_05.STL
- link Link_arm_l_06: geometry collision mesh filename=package://TR5/meshes/Link_arm_l_06.STL; visual mesh filename=package://TR5/meshes/Link_arm_l_06.STL
- link Link_arm_l_07: geometry collision mesh filename=package://TR5/meshes/Link_arm_l_07.STL; visual mesh filename=package://TR5/meshes/Link_arm_l_07.STL
- link Link_arm_r_01: geometry collision mesh filename=package://TR5/meshes/Link_arm_r_01.STL; visual mesh filename=package://TR5/meshes/Link_arm_r_01.STL
- link Link_arm_r_02: geometry collision mesh filename=package://TR5/meshes/Link_arm_r_02.STL; visual mesh filename=package://TR5/meshes/Link_arm_r_02.STL
- link Link_arm_r_03: geometry collision mesh filename=package://TR5/meshes/Link_arm_r_03.STL; visual mesh filename=package://TR5/meshes/Link_arm_r_03.STL
- link Link_arm_r_04: geometry collision mesh filename=package://TR5/meshes/Link_arm_r_04.STL; visual mesh filename=package://TR5/meshes/Link_arm_r_04.STL
- link Link_arm_r_05: geometry collision mesh filename=package://TR5/meshes/Link_arm_r_05.STL; visual mesh filename=package://TR5/meshes/Link_arm_r_05.STL
- link Link_arm_r_06: geometry collision mesh filename=package://TR5/meshes/Link_arm_r_06.STL; visual mesh filename=package://TR5/meshes/Link_arm_r_06.STL
- link Link_arm_r_07: geometry collision mesh filename=package://TR5/meshes/Link_arm_r_07.STL; visual mesh filename=package://TR5/meshes/Link_arm_r_07.STL
- link Link_head_pitch: geometry collision mesh filename=package://TR5/meshes/Link_head_pitch.STL; visual mesh filename=package://TR5/meshes/Link_head_pitch.STL
- link Link_head_yaw: geometry collision mesh filename=package://TR5/meshes/Link_head_yaw.STL; visual mesh filename=package://TR5/meshes/Link_head_yaw.STL
- link Link_hip_l_pitch: geometry collision mesh filename=package://TR5/meshes/Link_hip_l_pitch.STL; visual mesh filename=package://TR5/meshes/Link_hip_l_pitch.STL
- link Link_hip_l_roll: geometry collision mesh filename=package://TR5/meshes/Link_hip_l_roll.STL; visual mesh filename=package://TR5/meshes/Link_hip_l_roll.STL
- link Link_hip_l_yaw: geometry collision mesh filename=package://TR5/meshes/Link_hip_l_yaw.STL; visual mesh filename=package://TR5/meshes/Link_hip_l_yaw.STL
- link Link_hip_r_pitch: geometry collision mesh filename=package://TR5/meshes/Link_hip_r_pitch.STL; visual mesh filename=package://TR5/meshes/Link_hip_r_pitch.STL
- link Link_hip_r_roll: geometry collision mesh filename=package://TR5/meshes/Link_hip_r_roll.STL; visual mesh filename=package://TR5/meshes/Link_hip_r_roll.STL
- link Link_hip_r_yaw: geometry collision mesh filename=package://TR5/meshes/Link_hip_r_yaw.STL; visual mesh filename=package://TR5/meshes/Link_hip_r_yaw.STL
- link Link_knee_l_pitch: geometry collision mesh filename=package://TR5/meshes/Link_knee_l_pitch.STL; visual mesh filename=package://TR5/meshes/Link_knee_l_pitch.STL
- link Link_knee_r_pitch: geometry collision mesh filename=package://TR5/meshes/Link_knee_r_pitch.STL; visual mesh filename=package://TR5/meshes/Link_knee_r_pitch.STL
- link Link_waist_roll: geometry collision mesh filename=package://TR5/meshes/Link_waist_roll.STL; visual mesh filename=package://TR5/meshes/Link_waist_roll.STL
- link Link_waist_yaw: geometry collision mesh filename=package://TR5/meshes/Link_waist_yaw.STL; visual mesh filename=package://TR5/meshes/Link_waist_yaw.STL
- link base_link: geometry collision mesh filename=package://TR5/meshes/base_link.STL; visual mesh filename=package://TR5/meshes/base_link.STL
